Commit message: running the standalone model for the avatar

File: avater/avatar_drake_detailed_hand.urdf (robot description, URDF)
Before this commit: robot avatar, 100 links, 99 joints
Links:
- link gofa1_base: geometry collision mesh filename=avatar_model/abb_gofa/meshes/collision_obj/base.obj; visual mesh filename=avatar_model/abb_gofa/meshes/visual_obj/base.obj
- link gofa1_link_1: geometry collision mesh filename=avatar_model/abb_gofa/meshes/collision_obj/link_1.obj; visual mesh filename=avatar_model/abb_gofa/meshes/visual_obj/link_1.obj
- link gofa1_link_2: geometry collision mesh filename=avatar_model/abb_gofa/meshes/collision_obj/link_2.obj; visual mesh filename=avatar_model/abb_gofa/meshes/visual_obj/link_2.obj
- link gofa1_link_3: geometry collision mesh filename=avatar_model/abb_gofa/meshes/collision_obj/link_3.obj; visual mesh filename=avatar_model/abb_gofa/meshes/visual_obj/link_3.obj
- link gofa1_link_4: geometry collision mesh filename=avatar_model/abb_gofa/meshes/collision_obj/link_4.obj; visual mesh filename=avatar_model/abb_gofa/meshes/visual_obj/link_4.obj
- link gofa1_link_5: geometry collision mesh filename=avatar_model/abb_gofa/meshes/collision_obj/link_5.obj; visual mesh filename=avatar_model/abb_gofa/meshes/visual_obj/link_5.obj
- link gofa1_link_6: geometry collision mesh filename=avatar_model/abb_gofa/meshes/collision_obj/link_6.obj; visual mesh filename=avatar_model/abb_gofa/meshes/visual_obj/link_6.obj
- link gofa2_base: geometry collision mesh filename=avatar_model/abb_gofa/meshes/collision_obj/base.obj; visual mesh filename=avatar_model/abb_gofa/meshes/visual_obj/base.obj
- link gofa2_link_1: geometry collision mesh filename=avatar_model/abb_gofa/meshes/collision_obj/link_1.obj; visual mesh filename=avatar_model/abb_gofa/meshes/visual_obj/link_1.obj
- link gofa2_link_2: geometry collision mesh filename=avatar_model/abb_gofa/meshes/collision_obj/link_2.obj; visual mesh filename=avatar_model/abb_gofa/meshes/visual_obj/link_2.obj
- link gofa2_link_3: geometry collision mesh filename=avatar_model/abb_gofa/meshes/collision_obj/link_3.obj; visual mesh filename=avatar_model/abb_gofa/meshes/visual_obj/link_3.obj
- link gofa2_link_4: geometry collision mesh filename=avatar_model/abb_gofa/meshes/collision_obj/link_4.obj; visual mesh filename=avatar_model/abb_gofa/meshes/visual_obj/link_4.obj
- link gofa2_link_5: geometry collision mesh filename=avatar_model/abb_gofa/meshes/collision_obj/link_5.obj; visual mesh filename=avatar_model/abb_gofa/meshes/visual_obj/link_5.obj
- link gofa2_link_6: geometry collision mesh filename=avatar_model/abb_gofa/meshes/collision_obj/link_6.obj; visual mesh filename=avatar_model/abb_gofa/meshes/visual_obj/link_6.obj
- link lh_ffdistal: geometry collision mesh filename=avatar_model/shadow_hand/meshes_drake/f_distal_bt_sp.obj scale=0.001 0.001 0.001; visual mesh filename=avatar_model/shadow_hand/meshes_drake/f_distal_bt_sp.obj scale=0.001 0.001 0.001
- link lh_ffknuckle: geometry collision cylinder length=0.014 radius=0.007; visual mesh filename=avatar_model/shadow_hand/meshes_drake/f_knuckle_e3m5.obj scale=0.001 0.001 0.001
- link lh_ffmiddle: geometry collision cylinder length=0.025 radius=0.007; collision sphere radius=0.007
- link lh_ffproximal: geometry collision cylinder length=0.040 radius=0.007; visual mesh filename=avatar_model/shadow_hand/meshes_drake/f_proximal_e3m5.obj scale=0.001 0.001 0.001
- link lh_forearm: geometry collision box size=0.07 0.07 0.07; collision mesh filename=avatar_model/shadow_hand/meshes_drake/forearm_collision_e3m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 scale=0.001 0.001 0.001
- link lh_lfdistal: geometry collision mesh filename=avatar_model/shadow_hand/meshes_drake/f_distal_bt_sp.obj scale=0.001 0.001 0.001; visual mesh filename=avatar_model/shadow_hand/meshes_drake/f_distal_bt_sp.obj scale=0.001 0.001 0.001
- link lh_lfknuckle: geometry collision cylinder length=0.014 radius=0.007; visual mesh filename=avatar_model/shadow_hand/meshes_drake/f_knuckle_e3m5.obj scale=0.001 0.001 0.001
- link lh_lfmetacarpal: geometry collision box size=0.018 0.024 0.040; visual mesh filename=avatar_model/shadow_hand/meshes_drake/lf_metacarpal_e3m5.obj scale=0.001 0.001 0.001
- link lh_lfmiddle: geometry collision cylinder length=0.025 radius=0.007; collision sphere radius=0.007
- link lh_lfproximal: geometry collision cylinder length=0.040 radius=0.007; visual mesh filename=avatar_model/shadow_hand/meshes_drake/f_proximal_e3m5.obj scale=0.001 0.001 0.001
- link lh_mfdistal: geometry collision mesh filename=avatar_model/shadow_hand/meshes_drake/f_distal_bt_sp.obj scale=0.001 0.001 0.001; visual mesh filename=avatar_model/shadow_hand/meshes_drake/f_distal_bt_sp.obj scale=0.001 0.001 0.001
- link lh_mfknuckle: geometry collision cylinder length=0.014 radius=0.007; visual mesh filename=avatar_model/shadow_hand/meshes_drake/f_knuckle_e3m5.obj scale=0.001 0.001 0.001
- link lh_mfmiddle: geometry collision cylinder length=0.025 radius=0.007; collision sphere radius=0.007
- link lh_mfproximal: geometry collision cylinder length=0.040 radius=0.007; visual mesh filename=avatar_model/shadow_hand/meshes_drake/f_proximal_e3m5.obj scale=0.001 0.001 0.001
- link lh_palm: geometry collision box size=0.018 0.024 0.004; collision box size=0.020 0.024 0.040
- link lh_rfdistal: geometry collision mesh filename=avatar_model/shadow_hand/meshes_drake/f_distal_bt_sp.obj scale=0.001 0.001 0.001; visual mesh filename=avatar_model/shadow_hand/meshes_drake/f_distal_bt_sp.obj scale=0.001 0.001 0.001
- link lh_rfknuckle: geometry collision cylinder length=0.014 radius=0.007; visual mesh filename=avatar_model/shadow_hand/meshes_drake/f_knuckle_e3m5.obj scale=0.001 0.001 0.001
- link lh_rfmiddle: geometry collision cylinder length=0.025 radius=0.007; collision sphere radius=0.007
- link lh_rfproximal: geometry collision cylinder length=0.040 radius=0.007; visual mesh filename=avatar_model/shadow_hand/meshes_drake/f_proximal_e3m5.obj scale=0.001 0.001 0.001
- link lh_thdistal: geometry collision mesh filename=avatar_model/shadow_hand/meshes_drake/th_distal_bt_sp.obj scale=0.001 0.001 0.001; visual mesh filename=avatar_model/shadow_hand/meshes_drake/th_distal_bt_sp.obj scale=0.001 0.001 0.001
- link lh_thmiddle: geometry collision cylinder length=0.014 radius=0.010; collision cylinder length=0.018 radius=0.011
- link lh_thproximal: geometry collision cylinder length=0.018 radius=0.012; visual mesh filename=avatar_model/shadow_hand/meshes_drake/th_proximal_e3m5.obj scale=0.001 0.001 0.001
- link lh_wrist: geometry collision box size=0.027 0.018 0.010; collision box size=0.027 0.018 0.010
- link rh_ffdistal: geometry collision mesh filename=avatar_model/shadow_hand/meshes_drake/f_distal_bt_sp.obj scale=0.001 0.001 0.001; visual mesh filename=avatar_model/shadow_hand/meshes_drake/f_distal_bt_sp.obj scale=0.001 0.001 0.001
- link rh_ffknuckle: geometry collision cylinder length=0.014 radius=0.007; visual mesh filename=avatar_model/shadow_hand/meshes_drake/f_knuckle_e3m5.obj scale=0.001 0.001 0.001
- link rh_ffmiddle: geometry collision cylinder length=0.025 radius=0.007; collision sphere radius=0.007
- link rh_ffproximal: geometry collision cylinder length=0.040 radius=0.007; visual mesh filename=avatar_model/shadow_hand/meshes_drake/f_proximal_e3m5.obj scale=0.001 0.001 0.001
- link rh_forearm: geometry collision box size=0.07 0.07 0.07; collision mesh filename=avatar_model/shadow_hand/meshes_drake/forearm_collision_e3m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 scale=0.001 0.001 0.001
- link rh_lfdistal: geometry collision mesh filename=avatar_model/shadow_hand/meshes_drake/f_distal_bt_sp.obj scale=0.001 0.001 0.001; visual mesh filename=avatar_model/shadow_hand/meshes_drake/f_distal_bt_sp.obj scale=0.001 0.001 0.001
- link rh_lfknuckle: geometry collision cylinder length=0.014 radius=0.007; visual mesh filename=avatar_model/shadow_hand/meshes_drake/f_knuckle_e3m5.obj scale=0.001 0.001 0.001
- link rh_lfmetacarpal: geometry collision box size=0.018 0.024 0.040; visual mesh filename=avatar_model/shadow_hand/meshes_drake/lf_metacarpal_e3m5.obj scale=0.001 0.001 0.001
- link rh_lfmiddle: geometry collision cylinder length=0.025 radius=0.007; collision sphere radius=0.007
- link rh_lfproximal: geometry collision cylinder length=0.040 radius=0.007; visual mesh filename=avatar_model/shadow_hand/meshes_drake/f_proximal_e3m5.obj scale=0.001 0.001 0.001
- link rh_mfdistal: geometry collision mesh filename=avatar_model/shadow_hand/meshes_drake/f_distal_bt_sp.obj scale=0.001 0.001 0.001; visual mesh filename=avatar_model/shadow_hand/meshes_drake/f_distal_bt_sp.obj scale=0.001 0.001 0.001
- link rh_mfknuckle: geometry collision cylinder length=0.014 radius=0.007; visual mesh filename=avatar_model/shadow_hand/meshes_drake/f_knuckle_e3m5.obj scale=0.001 0.001 0.001
- link rh_mfmiddle: geometry collision cylinder length=0.025 radius=0.007; collision sphere radius=0.007
- link rh_mfproximal: geometry collision cylinder length=0.040 radius=0.007; visual mesh filename=avatar_model/shadow_hand/meshes_drake/f_proximal_e3m5.obj scale=0.001 0.001 0.001
- link rh_palm: geometry collision box size=0.018 0.024 0.004; collision box size=0.020 0.024 0.040
- link rh_rfdistal: geometry collision mesh filename=avatar_model/shadow_hand/meshes_drake/f_distal_bt_sp.obj scale=0.001 0.001 0.001; visual mesh filename=avatar_model/shadow_hand/meshes_drake/f_distal_bt_sp.obj scale=0.001 0.001 0.001
- link rh_rfknuckle: geometry collision cylinder length=0.014 radius=0.007; visual mesh filename=avatar_model/shadow_hand/meshes_drake/f_knuckle_e3m5.obj scale=0.001 0.001 0.001
- link rh_rfmiddle: geometry collision cylinder length=0.025 radius=0.007; collision sphere radius=0.007
- link rh_rfproximal: geometry collision cylinder length=0.040 radius=0.007; visual mesh filename=avatar_model/shadow_hand/meshes_drake/f_proximal_e3m5.obj scale=0.001 0.001 0.001
- link rh_thdistal: geometry collision mesh filename=avatar_model/shadow_hand/meshes_drake/th_distal_bt_sp.obj scale=0.001 0.001 0.001; visual mesh filename=avatar_model/shadow_hand/meshes_drake/th_distal_bt_sp.obj scale=0.001 0.001 0.001
- link rh_thmiddle: geometry collision cylinder length=0.014 radius=0.010; collision cylinder length=0.018 radius=0.011
- link rh_thproximal: geometry collision cylinder length=0.018 radius=0.012; visual mesh filename=avatar_model/shadow_hand/meshes_drake/th_proximal_e3m5.obj scale=0.001 0.001 0.001
- link rh_wrist: geometry collision box size=0.027 0.018 0.010; collision box size=0.027 0.018 0.010
- link xarm6_link1: geometry collision mesh filename=avatar_model/xarm/visual_obj/link1.obj; visual mesh filename=avatar_model/xarm/visual_obj/link1.obj
- link xarm6_link2: geometry collision mesh filename=avatar_model/xarm/visual_obj/link2.obj; visual mesh filename=avatar_model/xarm/visual_obj/link2.obj
- link xarm6_link3: geometry collision mesh filename=avatar_model/xarm/visual_obj/link3.obj; visual mesh filename=avatar_model/xarm/visual_obj/link3.obj
- link xarm6_link4: geometry collision mesh filename=avatar_model/xarm/visual_obj/link4.obj; visual mesh filename=avatar_model/xarm/visual_obj/link4.obj
- link xarm6_link5: geometry collision mesh filename=avatar_model/xarm/visual_obj/link5.obj; visual mesh filename=avatar_model/xarm/visual_obj/link5.obj
- link xarm6_link6: geometry collision mesh filename=avatar_model/xarm/end_tool/collision/end_tool.obj; visual mesh filename=avatar_model/xarm/visual_obj/link6.obj
- link xarm6_link_base: geometry collision mesh filename=avatar_model/xarm/visual_obj/base.obj; visual mesh filename=avatar_model/xarm/visual_obj/base.obj
Joints:
- removed joint gofa1_base_workspace_joint
- added joint gofa1_base_link: type fixed, parent gofa1_workspace, child gofa1_base_link, origin xyz=0.0 0.0 0.095 rpy=0.0 -0.523599 0.0
