Commit message: running the standalone model for the avatar

File: avater/avatar_genesis.urdf (robot description, URDF)
Before this commit: robot avatar, 100 links, 99 joints
Links:
- link gofa1_base: geometry collision mesh filename=avatar_model/abb_gofa/meshes/collision_stl/base.STL; visual mesh filename=avatar_model/abb_gofa/meshes/visual_stl/base.STL
- link gofa1_link_1: geometry collision mesh filename=avatar_model/abb_gofa/meshes/collision_stl/link_1.STL; visual mesh filename=avatar_model/abb_gofa/meshes/visual_stl/link_1.STL
- link gofa1_link_2: geometry collision mesh filename=avatar_model/abb_gofa/meshes/collision_stl/link_2.STL; visual mesh filename=avatar_model/abb_gofa/meshes/visual_stl/link_2.STL
- link gofa1_link_3: geometry collision mesh filename=avatar_model/abb_gofa/meshes/collision_stl/link_3.STL; visual mesh filename=avatar_model/abb_gofa/meshes/visual_stl/link_3.STL
- link gofa1_link_4: geometry collision mesh filename=avatar_model/abb_gofa/meshes/collision_stl/link_4.STL; visual mesh filename=avatar_model/abb_gofa/meshes/visual_stl/link_4.STL
- link gofa1_link_5: geometry collision mesh filename=avatar_model/abb_gofa/meshes/collision_stl/link_5.STL; visual mesh filename=avatar_model/abb_gofa/meshes/visual_stl/link_5.STL
- link gofa1_link_6: geometry collision mesh filename=avatar_model/abb_gofa/meshes/collision_stl/link_6.STL; visual mesh filename=avatar_model/abb_gofa/meshes/visual_stl/link_6.STL
- link gofa2_base: geometry collision mesh filename=avatar_model/abb_gofa/meshes/collision_stl/base.STL; visual mesh filename=avatar_model/abb_gofa/meshes/visual_stl/base.STL
- link gofa2_link_1: geometry collision mesh filename=avatar_model/abb_gofa/meshes/collision_stl/link_1.STL; visual mesh filename=avatar_model/abb_gofa/meshes/visual_stl/link_1.STL
- link gofa2_link_2: geometry collision mesh filename=avatar_model/abb_gofa/meshes/collision_stl/link_2.STL; visual mesh filename=avatar_model/abb_gofa/meshes/visual_stl/link_2.STL
- link gofa2_link_3: geometry collision mesh filename=avatar_model/abb_gofa/meshes/collision_stl/link_3.STL; visual mesh filename=avatar_model/abb_gofa/meshes/visual_stl/link_3.STL
- link gofa2_link_4: geometry collision mesh filename=avatar_model/abb_gofa/meshes/collision_stl/link_4.STL; visual mesh filename=avatar_model/abb_gofa/meshes/visual_stl/link_4.STL
- link gofa2_link_5: geometry collision mesh filename=avatar_model/abb_gofa/meshes/collision_stl/link_5.STL; visual mesh filename=avatar_model/abb_gofa/meshes/visual_stl/link_5.STL
- link gofa2_link_6: geometry collision mesh filename=avatar_model/abb_gofa/meshes/collision_stl/link_6.STL; visual mesh filename=avatar_model/abb_gofa/meshes/visual_stl/link_6.STL
- link lh_ffdistal: geometry collision mesh filename=avatar_model/shadow_hand/meshes/collision_stl/finger_distal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 scale=0.001 0.001 0.001; visual mesh filename=avatar_model/shadow_hand/meshes/collision_stl/finger_distal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 scale=0.001 0.001 0.001
- link lh_ffknuckle: geometry collision cylinder length=0.014 radius=0.007; visual mesh filename=avatar_model/shadow_hand/meshes/collision_stl/knuckle.stl scale=0.001 0.001 0.001
- link lh_ffmiddle: geometry collision cylinder length=0.025 radius=0.007; collision sphere radius=0.007
- link lh_ffproximal: geometry collision cylinder length=0.040 radius=0.007; visual mesh filename=avatar_model/shadow_hand/meshes/collision_stl/finger_proxim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 scale=0.001 0.001 0.001
- link lh_forearm: geometry collision box size=0.07 0.07 0.07; collision mesh filename=avatar_model/shadow_hand/meshes/collision_stl/forearm.stl scale=0.001 0.001 0.001
- link lh_lfdistal: geometry collision mesh filename=avatar_model/shadow_hand/meshes/collision_stl/finger_distal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 scale=0.001 0.001 0.001; visual mesh filename=avatar_model/shadow_hand/meshes/collision_stl/finger_distal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 scale=0.001 0.001 0.001
- link lh_lfknuckle: geometry collision cylinder length=0.014 radius=0.007; visual mesh filename=avatar_model/shadow_hand/meshes/collision_stl/knuckle.stl scale=0.001 0.001 0.001
- link lh_lfmetacarpal: geometry collision box size=0.018 0.024 0.040; visual mesh filename=avatar_model/shadow_hand/meshes/collision_stl/metacarpal.stl scale=0.001 0.001 0.001
- link lh_lfmiddle: geometry collision cylinder length=0.025 radius=0.007; collision sphere radius=0.007
- link lh_lfproximal: geometry collision cylinder length=0.040 radius=0.007; visual mesh filename=avatar_model/shadow_hand/meshes/collision_stl/finger_proxim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 scale=0.001 0.001 0.001
- link lh_mfdistal: geometry collision mesh filename=avatar_model/shadow_hand/meshes/collision_stl/finger_distal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 scale=0.001 0.001 0.001; visual mesh filename=avatar_model/shadow_hand/meshes/collision_stl/finger_distal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 scale=0.001 0.001 0.001
- link lh_mfknuckle: geometry collision cylinder length=0.014 radius=0.007; visual mesh filename=avatar_model/shadow_hand/meshes/collision_stl/knuckle.stl scale=0.001 0.001 0.001
- link lh_mfmiddle: geometry collision cylinder length=0.025 radius=0.007; collision sphere radius=0.007
- link lh_mfproximal: geometry collision cylinder length=0.040 radius=0.007; visual mesh filename=avatar_model/shadow_hand/meshes/collision_stl/finger_proxim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 scale=0.001 0.001 0.001
- link lh_palm: geometry collision box size=0.018 0.024 0.004; collision box size=0.020 0.024 0.040
- link lh_rfdistal: geometry collision mesh filename=avatar_model/shadow_hand/meshes/collision_stl/finger_distal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 scale=0.001 0.001 0.001; visual mesh filename=avatar_model/shadow_hand/meshes/collision_stl/finger_distal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 scale=0.001 0.001 0.001
- link lh_rfknuckle: geometry collision cylinder length=0.014 radius=0.007; visual mesh filename=avatar_model/shadow_hand/meshes/collision_stl/knuckle.stl scale=0.001 0.001 0.001
- link lh_rfmiddle: geometry collision cylinder length=0.025 radius=0.007; collision sphere radius=0.007
- link lh_rfproximal: geometry collision cylinder length=0.040 radius=0.007; visual mesh filename=avatar_model/shadow_hand/meshes/collision_stl/finger_proxim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 scale=0.001 0.001 0.001
- link lh_thdistal: geometry collision mesh filename=avatar_model/shadow_hand/meshes/collision_stl/thumb_distal.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 scale=0.001 0.001 0.001; visual mesh filename=avatar_model/shadow_hand/meshes/collision_stl/thumb_distal.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 scale=0.001 0.001 0.001
- link lh_thmiddle: geometry collision cylinder length=0.014 radius=0.010; collision cylinder length=0.018 radius=0.011
- link lh_thproximal: geometry collision cylinder length=0.018 radius=0.012; visual mesh filename=avatar_model/shadow_hand/meshes/collision_stl/thumb_proxima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 scale=0.001 0.001 0.001
- link lh_wrist: geometry collision box size=0.027 0.018 0.010; collision box size=0.027 0.018 0.010
- link rh_ffdistal: geometry collision mesh filename=avatar_model/shadow_hand/meshes/collision_stl/finger_distal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 scale=0.001 0.001 0.001; visual mesh filename=avatar_model/shadow_hand/meshes/collision_stl/finger_distal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 scale=0.001 0.001 0.001
- link rh_ffknuckle: geometry collision cylinder length=0.014 radius=0.007; visual mesh filename=avatar_model/shadow_hand/meshes/collision_stl/knuckle.stl scale=0.001 0.001 0.001
- link rh_ffmiddle: geometry collision cylinder length=0.025 radius=0.007; collision sphere radius=0.007
- link rh_ffproximal: geometry collision cylinder length=0.040 radius=0.007; visual mesh filename=avatar_model/shadow_hand/meshes/collision_stl/finger_proxim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 scale=0.001 0.001 0.001
- link rh_forearm: geometry collision box size=0.07 0.07 0.07; collision mesh filename=avatar_model/shadow_hand/meshes/collision_stl/forearm.stl scale=0.001 0.001 0.001
- link rh_lfdistal: geometry collision mesh filename=avatar_model/shadow_hand/meshes/collision_stl/finger_distal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 scale=0.001 0.001 0.001; visual mesh filename=avatar_model/shadow_hand/meshes/collision_stl/finger_distal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 scale=0.001 0.001 0.001
- link rh_lfknuckle: geometry collision cylinder length=0.014 radius=0.007; visual mesh filename=avatar_model/shadow_hand/meshes/collision_stl/knuckle.stl scale=0.001 0.001 0.001
- link rh_lfmetacarpal: geometry collision box size=0.018 0.024 0.040; visual mesh filename=avatar_model/shadow_hand/meshes/collision_stl/metacarpal.stl scale=0.001 0.001 0.001
- link rh_lfmiddle: geometry collision cylinder length=0.025 radius=0.007; collision sphere radius=0.007
- link rh_lfproximal: geometry collision cylinder length=0.040 radius=0.007; visual mesh filename=avatar_model/shadow_hand/meshes/collision_stl/finger_proxim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 scale=0.001 0.001 0.001
- link rh_mfdistal: geometry collision mesh filename=avatar_model/shadow_hand/meshes/collision_stl/finger_distal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 scale=0.001 0.001 0.001; visual mesh filename=avatar_model/shadow_hand/meshes/collision_stl/finger_distal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 scale=0.001 0.001 0.001
- link rh_mfknuckle: geometry collision cylinder length=0.014 radius=0.007; visual mesh filename=avatar_model/shadow_hand/meshes/collision_stl/knuckle.stl scale=0.001 0.001 0.001
- link rh_mfmiddle: geometry collision cylinder length=0.025 radius=0.007; collision sphere radius=0.007
- link rh_mfproximal: geometry collision cylinder length=0.040 radius=0.007; visual mesh filename=avatar_model/shadow_hand/meshes/collision_stl/finger_proxim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 scale=0.001 0.001 0.001
- link rh_palm: geometry collision box size=0.018 0.024 0.004; collision box size=0.020 0.024 0.040
- link rh_rfdistal: geometry collision mesh filename=avatar_model/shadow_hand/meshes/collision_stl/finger_distal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 scale=0.001 0.001 0.001; visual mesh filename=avatar_model/shadow_hand/meshes/collision_stl/finger_distal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 scale=0.001 0.001 0.001
- link rh_rfknuckle: geometry collision cylinder length=0.014 radius=0.007; visual mesh filename=avatar_model/shadow_hand/meshes/collision_stl/knuckle.stl scale=0.001 0.001 0.001
- link rh_rfmiddle: geometry collision cylinder length=0.025 radius=0.007; collision sphere radius=0.007
- link rh_rfproximal: geometry collision cylinder length=0.040 radius=0.007; visual mesh filename=avatar_model/shadow_hand/meshes/collision_stl/finger_proxim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 scale=0.001 0.001 0.001
- link rh_thdistal: geometry collision mesh filename=avatar_model/shadow_hand/meshes/collision_stl/thumb_distal.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 scale=0.001 0.001 0.001; visual mesh filename=avatar_model/shadow_hand/meshes/collision_stl/thumb_distal.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 scale=0.001 0.001 0.001
- link rh_thmiddle: geometry collision cylinder length=0.014 radius=0.010; collision cylinder length=0.018 radius=0.011
- link rh_thproximal: geometry collision cylinder length=0.018 radius=0.012; visual mesh filename=avatar_model/shadow_hand/meshes/collision_stl/thumb_proxima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 scale=0.001 0.001 0.001
- link rh_wrist: geometry collision box size=0.027 0.018 0.010; collision box size=0.027 0.018 0.010
- link xarm6_link1: geometry collision mesh filename=avatar_model/xarm/visual_stl/link1.stl; visual mesh filename=avatar_model/xarm/visual_stl/link1.stl
- link xarm6_link2: geometry collision mesh filename=avatar_model/xarm/visual_stl/link2.stl; visual mesh filename=avatar_model/xarm/visual_stl/link2.stl
- link xarm6_link3: geometry collision mesh filename=avatar_model/xarm/visual_stl/link3.stl; visual mesh filename=avatar_model/xarm/visual_stl/link3.stl
- link xarm6_link4: geometry collision mesh filename=avatar_model/xarm/visual_stl/link4.stl; visual mesh filename=avatar_model/xarm/visual_stl/link4.stl
- link xarm6_link5: geometry collision mesh filename=avatar_model/xarm/visual_stl/link5.stl; visual mesh filename=avatar_model/xarm/visual_stl/link5.stl
- link xarm6_link6: geometry collision mesh filename=avatar_model/xarm/end_tool/collision/end_tool.stl; visual mesh filename=avatar_model/xarm/visual_stl/link6.stl
- link xarm6_link_base: geometry collision mesh filename=avatar_model/xarm/visual_stl/base.stl; visual mesh filename=avatar_model/xarm/visual_stl/base.stl
